File: auto flash.brd (EAGLE design)
At the start: 22.9 x 24.1 mm, 8 parts, among them T1 s8050, T2 s8050

Commit message: add esp-12, esp-07 adapter
Parts:
- JP1: value (none) -> cp2102
- JP2: value (none) -> ESP-01
- R1, R2: value 10k -> 12k
Connections:
- net N$10 renamed ESP-01
Changed lines of the file:
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@@
 </autorouter>
 <elements>
-<element name="JP1" library="pinhead" package="1X07/90" value="" x="54.61" y="71.12" rot="MR0"/>
-<element name="JP2" library="pinhead" package="2X04" value="" x="50.8" y="53.34" rot="MR180"/>
-<element name="R1" library="SparkFun-Resistors" package="0805" value="10k" x="50.8" y="58.42">
+<element name="JP1" library="pinhead" package="1X07/90" value="cp2102" x="54.61" y="71.12" rot="MR0"/>
+<element name="JP2" library="pinhead" package="2X04" value="ESP-01" x="50.8" y="53.34" rot="MR180"/>
+<element name="R1" library="SparkFun-Resistors" package="0805" value="12k" x="50.8" y="58.42">
 <attribute name="PROD_ID" value="RES-11622" x="50.8" y="58.42" size="1.778" layer="27" display="off"/>
 </element>
-<element name="R2" library="SparkFun-Resistors" package="0805" value="10k" x="50.8" y="64.77" rot="R180">
+<element name="R2" library="SparkFun-Resistors" package="0805" value="12k" x="50.8" y="64.77" rot="R180">
 <attribute name="PROD_ID" value="RES-11622" x="50.8" y="64.77" size="1.778" layer="27" rot="R180" display="off"/>
 </element>
@@
 <wire x1="60.96" y1="54.61" x2="60.96" y2="55.3212" width="0" layer="19" extent="1-16"/>
 </signal>
-<signal name="N$10">
+<signal name="ESP-01">
 <contactref element="JP1" pad="4"/>
 <contactref element="JP2" pad="1"/>
